File: Electrium-Mobility-KiCad.kicad_sch (KiCad schematic)
At the start: 25 parts, among them M1 3V 75mA, Q1 NMOS, SW1 SW_Push, SW2 SW_Push, U1 ESP32-WROOM-32E, U2 LCD-016N002L, U3 TPB4056A20-ES1R

Commit message: Fix Schematic Signed-off-by: David Xu <131167198+DavidX787@users.noreply.github.com>
Parts:
- C1: value C -> 10 uF/16V
- C2: value C -> 0.1 uF / 16V
- R IMIN: value tbd -> 16000 Ohms
- R IREF: value ~ -> 4k Ohms
- R6: value ??? Ohms -> 330 Ohms
- R7: value R_Small_US -> 330 Ohms
Connections:
- net Earth is gone; now on net GND: AH8501-FDC-7 HES1.5 (GND), BT1.2 (-), C2.2, D1.1 (K), D2.1 (K), D3.2 (A), R IMIN.2, R IREF.2, RV1.1, SW1.2, SW2.2, U1.1 (GND), U1.15 (GND), U1.38 (GND), U1.39 (GND), U2.1 (VSS), U2.16 (K), U2.5 (R/~{W}), U2.K1, U2.K2, U3.5 (GND), U3.9 (GND)
- net at Q1.1 (D), Q1.2 (G), U1.25 (IO0): now also M1.1 (+)
- net GND: now reaches U3.4 (*EN)
- net GND: now also M1.2 (-)
Changed lines of the file:
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@@
+	(wire
+		(pts
+			(xy 22.86 99.06) (xy 22.86 101.6)
+		)
+		(stroke
+			(width 0)
+			(type default)
+		)
+	)
+	(wire
+		(pts
+			(xy 194.31 67.31) (xy 194.31 68.58)
+		)
+		(stroke
+			(width 0)
+			(type default)
+		)
+	)
+	(wire
+		(pts
+			(xy 124.46 110.49) (xy 124.46 146.05)
+		)
+		(stroke
+			(width 0)
+			(type default)
+		)
+	)
+	(wire
+		(pts
+			(xy 171.45 156.21) (xy 171.45 158.75)
+		)
+		(stroke
+			(width 0)
+			(type default)
+		)
+	)
+	(wire
+		(pts
+			(xy 152.4 146.05) (xy 152.4 158.75)
+		)
+		(stroke
+			(width 0)
+			(type default)
+		)
+	)
+	(wire
+		(pts
+			(xy 167.64 110.49) (xy 234.95 110.49)
+		)
+		(stroke
+			(width 0)
+			(type default)
+		)
+	)
+	(wire
+		(pts
+			(xy 22.86 87.63) (xy 22.86 91.44)
+		)
+		(stroke
+			(width 0)
+			(type default)
+		)
+	)
+	(wire
+		(pts
+			(xy 109.22 99.06) (xy 109.22 100.33)
+		)
+		(stroke
+			(width 0)
+			(type default)
+		)
+	)
 	(wire
 		(pts
@@
 	(wire
 		(pts
-			(xy 22.86 99.06) (xy 22.86 101.6)
+			(xy 31.75 96.52) (xy 31.75 99.06)
 		)
 		(stroke
@@
 	(wire
 		(pts
-			(xy 194.31 67.31) (xy 194.31 68.58)
+			(xy 234.95 120.65) (xy 167.64 120.65)
 		)
 		(stroke
@@
 	(wire
 		(pts
-			(xy 124.46 110.49) (xy 124.46 146.05)
+			(xy 92.71 41.91) (xy 92.71 101.6)
 		)
 		(stroke
@@
 	(wire
 		(pts
-			(xy 171.45 156.21) (xy 171.45 158.75)
+			(xy 22.86 78.74) (xy 22.86 82.55)
 		)
 		(stroke
@@
 	(wire
 		(pts
-			(xy 152.4 146.05) (xy 152.4 158.75)
+			(xy 255.27 85.09) (xy 257.81 85.09)
 		)
 		(stroke
@@
 	(wire
 		(pts
-			(xy 167.64 110.49) (xy 234.95 110.49)
+			(xy 30.48 78.74) (xy 30.48 96.52)
 		)
 		(stroke
@@
 	(wire
 		(pts
-			(xy 22.86 87.63) (xy 22.86 91.44)
+			(xy 274.32 68.58) (xy 274.32 91.44)
 		)
 		(stroke
@@
 		)
 	)
-	(wire
-		(pts
-			(xy 109.22 99.06) (xy 109.22 100.33)
-		)
-		(stroke
-			(width 0)
-			(type default)
-		)
-	)
-	(wire
-		(pts
-			(xy 31.75 96.52) (xy 31.75 99.06)
-		)
-		(stroke
-			(width 0)
-			(type default)
-		)
-	)
-	(wire
-		(pts
-			(xy 234.95 120.65) (xy 167.64 120.65)
-		)
-		(stroke
-			(width 0)
-			(type default)
-		)
-	)
-	(wire
-		(pts
-			(xy 92.71 41.91) (xy 92.71 101.6)
-		)
-		(stroke
-			(width 0)
-			(type default)
-		)
-	)
-	(wire
-		(pts
-			(xy 22.86 78.74) (xy 22.86 82.55)
-		)
-		(stroke
-			(width 0)
-			(type default)
-		)
-	)
-	(wire
-		(pts
-			(xy 255.27 85.09) (xy 257.81 85.09)
-		)
-		(stroke
-			(width 0)
-			(type default)
-		)
-	)
-	(wire
-		(pts
-			(xy 30.48 78.74) (xy 30.48 96.52)
-		)
-		(stroke
-			(width 0)
-			(type default)
-		)
-	)
-	(wire
-		(pts
-			(xy 274.32 68.58) (xy 274.32 91.44)
-		)
-		(stroke
-			(width 0)
-			(type default)
-		)
-	)
 	(symbol
 		(lib_id "power:Earth")
@@
 		(on_board yes)
 		(dnp no)
-		(fields_autoplaced yes)
 		(property "Reference" "#PWR01"
 			(at 81.28 115.57 0)
@@
 			)
 		)
-		(property "Value" "Earth"
-			(at 81.28 114.3 0)
-			(effects
-				(font
-					(size 1.27 1.27)
-				)
+		(property "Value" "GND"
+			(at 79.248 113.538 0)
+			(effects
+				(font
+					(size 1.27 1.27)
+				)
+				(justify left)
 			)
 		)
@@
 			)
 		)
-		(property "Value" "??? Ohms"
+		(property "Value" "330 Ohms"
 			(at 14.986 82.042 0)
 			(effects
@@
 			)
 		)
-		(property "Value" "tbd"
+		(property "Value" "16000 Ohms"
 			(at 73.914 113.284 90)
 			(effects
@@
 		(on_board yes)
 		(dnp no)
-		(fields_autoplaced yes)
 		(property "Reference" "C2"
 			(at 88.9 104.1399 0)
@@
 			)
 		)
-		(property "Value" "C"
-			(at 88.9 106.6799 0)
+		(property "Value" "0.1 uF / 16V"
+			(at 89.408 107.696 0)
 			(effects
 				(font
@@
 		(on_board yes)
 		(dnp no)
-		(fields_autoplaced yes)
 		(property "Reference" "R IREF"
 			(at 77.47 100.33 90)
@@
 			)
 		)
-		(property "Value" "~"
-			(at 78.7399 101.6 0)
+		(property "Value" "4k Ohms"
+			(at 81.534 102.87 90)
 			(effects
 				(font
@@
 			)
 		)
-		(property "Value" "R_Small_US"
+		(property "Value" "330 Ohms"
 			(at 25.4 86.3599 0)
 			(effects
@@
 			)
 		)
-		(property "Value" "C"
+		(property "Value" "10 uF/16V"
 			(at 31.75 83.8199 0)
 			(effects
@@
 					(unit 1)
 				)
+			)
+		)
+	)
+	(symbol
+		(lib_id "power:Earth")
+		(at 31.75 106.68 0)
+		(unit 1)
+		(exclude_from_sim no)
+		(in_bom yes)
+		(on_board yes)
+		(dnp no)
+		(property "Reference" "#PWR06"
+			(at 31.75 113.03 0)
+			(effects
+				(font
+					(size 1.27 1.27)
+				)
+				(hide yes)
+			)
+		)
+		(property "Value" "GND"
+			(at 29.718 110.998 0)
+			(effects
+				(font
+					(size 1.27 1.27)
+				)
+				(justify left)
+			)
+		)
+		(property "Footprint" ""
+			(at 31.75 106.68 0)
+			(effects
+				(font
+					(size 1.27 1.27)
+				)
+				(hide yes)
+			)
+		)
+		(property "Datasheet" "~"
+			(at 31.75 106.68 0)
+			(effects
+				(font
+					(size 1.27 1.27)
+				)
+				(hide yes)
+			)
+		)
+		(property "Description" "Power symbol creates a global label with name \"Earth\""
+			(at 31.75 106.68 0)
+			(effects
+				(font
+					(size 1.27 1.27)
+				)
+				(hide yes)
+			)
+		)
+		(pin "1"
+		)
+		(instances
+			(project "Electrium-Mobility-KiCad"
+				(path "/77cfd6b1-cf11-45d1-96c8-b00f1af024ba"
+					(reference "#PWR06")
+					(unit 1)
+				)
